File: pcb/project/secondscreen/secondscreen.kicad_sch (KiCad schematic)
At the start: 0 parts

Commit message: update
Parts:
- added A1: RaspberryPi_Pico, Module:RaspberryPi_Pico_Common_Unspecified, symbol MCU_Module:RaspberryPi_Pico
- added BZ1: Buzzer, symbol Device:Buzzer
- added M1, M2: Motor_Servo, symbol Motor:Motor_Servo
- added U2: 64x32px_320x160mm_RGB_LED_Matrix, symbol HUB75_64x32px_320x160mm_RGBLEDMATRIX:64x32px_320x160mm_RGB_LED_Matrix
Connections:
- new net +3.3V: A1.36 (3V3), M1.2 (+), M2.2 (+)
- new net +5V/4A (batt): U2. (GND)
- new net A: A1.9 (GPIO6), U2.7 (A)
- new net B: A1.16 (GPIO12), U2.8 (B)
- new net B1: A1.5 (GPIO3), U2.3 (B1)
- new net B2: A1.7 (GPIO5), U2.6 (B2)
- new net Buzz1: A1.20 (GPIO15), BZ1.1 (+)
- new net C: A1.10 (GPIO7), U2.9 (C)
- new net CLK: A1.11 (GPIO8), U2.11 (CLK)
- new net D: A1.17 (GPIO13), U2.10 (D/GND)
- new net G1: A1.14 (GPIO10), U2.2 (G1)
- new net G2: A1.15 (GPIO11), U2.5 (G2)
- new net GND: A1.13 (GND), A1.18 (GND), A1.23 (GND), A1.28 (GND), A1.3 (GND), A1.33 (AGND), A1.38 (GND), A1.8 (GND), BZ1.2 (-), M1.3 (-), M2.3 (-), U2.14 (GND)
- new net GND (batt): U2. (GND)
- new net LAT: A1.19 (GPIO14), U2.12 (LAT)
- new net OE: A1.12 (GPIO9), U2.13 (OE)
- new net R1: A1.4 (GPIO2), U2.1 (R1)
- new net R2: A1.6 (GPIO4), U2.4 (R2)
- new net motor1GPIO: A1.1 (GPIO0), M1.1 (PWM)
- new net motor2GPIO: A1.2 (GPIO1), M2.1 (PWM)
